Commit message: feat: i dont want to write this -m stuff

File: universal_robots_ur5e/ur5e_orig.urdf (robot description, URDF)
Before this commit: robot ur5e, 11 links, 10 joints
Links:
- added link transformed_base_link
Joints:
- added joint global_transform: type fixed, parent base_link, child transformed_base_link, origin xyz=0 0 0 rpy=0 0 3.141592653589793
- joint shoulder_pan_joint: parent base_link -> transformed_base_link
